Commit message: Clean-up of URDF.
Some joints are commented out because pybullet caps the number of
DoFs at 128; this includes fixed joints.

File: assets/trex.urdf (robot description, URDF)
Before this commit: robot stan_t_rex, 134 links, 133 joints
Links:
- removed link root_link
- removed link vertebra_caudal_26_link
- removed link vertebra_caudal_27_link
- removed link vertebra_caudal_28_link
- removed link vertebra_caudal_29_link
- removed link vertebra_caudal_30_link
- removed link vertebra_caudal_31_link
- removed link vertebra_caudal_32_link
- removed link vertebra_caudal_33_link
- removed link vertebra_caudal_34_link
- removed link vertebra_caudal_35_link
- removed link vertebra_caudal_36_link
- removed link vertebra_caudal_37_link
- removed link vertebra_caudal_38_link
- removed link vertebra_caudal_39_link
- removed link vertebra_caudal_40_link
- removed link vertebra_caudal_41_link
- removed link vertebra_caudal_42_link
- removed link vertebra_caudal_43_link
- removed link vertebra_caudal_44_link
Joints:
- removed joint vertebra_caudal_26_joint
- removed joint vertebra_caudal_27_joint
- removed joint vertebra_caudal_28_joint
- removed joint vertebra_caudal_29_joint
- removed joint vertebra_caudal_30_joint
- removed joint vertebra_caudal_31_joint
- removed joint vertebra_caudal_32_joint
- removed joint vertebra_caudal_33_joint
- removed joint vertebra_caudal_34_joint
- removed joint vertebra_caudal_35_joint
- removed joint vertebra_caudal_36_joint
- removed joint vertebra_caudal_37_joint
- removed joint vertebra_caudal_38_joint
- removed joint vertebra_caudal_39_joint
- removed joint vertebra_caudal_40_joint
- removed joint vertebra_caudal_41_joint
- removed joint vertebra_caudal_42_joint
- removed joint vertebra_caudal_43_joint
- removed joint vertebra_caudal_44_joint
- removed joint vertebrae_sacral_joint
- joint vertebra_caudal_10_joint: limit lower=-0.3490658503988659 upper=-0.3490658503988659 effort=100.0 velocity=1.0 -> lower=-0.3490658503988659 upper=0.3490658503988659 effort=100.0 velocity=1.0

Commit message: Hacking to find a policy that will solve.
* Switched to elevating head.
* Messed with caudal_10_joint x->z rotation.
* Commanding only position now, removed stiffness.
* Tweaked cost-coefficients to penalize lifting most.

File: assets/trex.urdf (robot description, URDF)
Before this commit: robot stan_t_rex, 114 links, 113 joints
Joints:
- joint vertebra_caudal_10_joint: axis 1.0 0.0 0.0 -> 0.0 0.0 1.0; limit lower=-0.3490658503988659 upper=0.3490658503988659 effort=100.0 velocity=1.0 -> lower=-1.3490658503988659 upper=1.3490658503988659 effort=100.0 velocity=1.0
