Commit message: Convert to OBJ and remove collision from URDF.

File: assets/trex.urdf (robot description, URDF)
Before this commit: robot stan_t_rex, 114 links, 113 joints
Links:
- added link vertebra_caudal_26_link, mass 1.4905412197113037; visual mesh filename=meshes/vis_gorgo_haemal_arch_27.obj scale=1.0 1.0 1.0; visual mesh filename=meshes/vis_vertebra_caudal_26.obj scale=1.0 1.0 1.0
- added link vertebra_caudal_27_link, mass 1.2704788446426392; visual mesh filename=meshes/vis_gorgo_haemal_arch_28.obj scale=1.0 1.0 1.0; visual mesh filename=meshes/vis_vertebra_caudal_27.obj scale=1.0 1.0 1.0
- added link vertebra_caudal_28_link, mass 1.2707126140594482; visual mesh filename=meshes/vis_gorgo_haemal_arch_29.obj scale=1.0 1.0 1.0; visual mesh filename=meshes/vis_vertebra_caudal_28.obj scale=1.0 1.0 1.0
- added link vertebra_caudal_29_link, mass 0.8220692276954651; visual mesh filename=meshes/vis_gorgo_haemal_arch_30.obj scale=1.0 1.0 1.0; visual mesh filename=meshes/vis_vertebra_caudal_29.obj scale=1.0 1.0 1.0
- added link vertebra_caudal_30_link, mass 0.5576320886611938; visual mesh filename=meshes/vis_gorgo_haemal_arch_31.obj scale=1.0 1.0 1.0; visual mesh filename=meshes/vis_vertebra_caudal_30.obj scale=1.0 1.0 1.0
- added link vertebra_caudal_31_link, mass 0.5741740465164185; visual mesh filename=meshes/vis_gorgo_haemal_arch_32.obj scale=1.0 1.0 1.0; visual mesh filename=meshes/vis_vertebra_caudal_31.obj scale=1.0 1.0 1.0
- added link vertebra_caudal_32_link, mass 0.385939359664917; visual mesh filename=meshes/vis_gorgo_haemal_arch_33.obj scale=1.0 1.0 1.0; visual mesh filename=meshes/vis_vertebra_caudal_32.obj scale=1.0 1.0 1.0
- added link vertebra_caudal_33_link, mass 0.3329651653766632; visual mesh filename=meshes/vis_gorgo_haemal_arch_34.obj scale=1.0 1.0 1.0; visual mesh filename=meshes/vis_vertebra_caudal_33.obj scale=1.0 1.0 1.0
- added link vertebra_caudal_34_link, mass 0.23780474066734314; visual mesh filename=meshes/vis_vertebra_caudal_34.obj scale=1.0 1.0 1.0
- added link vertebra_caudal_35_link, mass 0.24401071667671204; visual mesh filename=meshes/vis_vertebra_caudal_35.obj scale=1.0 1.0 1.0
- added link vertebra_caudal_36_link, mass 0.1726621389389038; visual mesh filename=meshes/vis_vertebra_caudal_36.obj scale=1.0 1.0 1.0
- added link vertebra_caudal_37_link, mass 0.10794775933027267; visual mesh filename=meshes/vis_vertebra_caudal_37.obj scale=1.0 1.0 1.0
- added link vertebra_caudal_38_link, mass 0.0814909115433693; visual mesh filename=meshes/vis_vertebra_caudal_38.obj scale=1.0 1.0 1.0
- added link vertebra_caudal_39_link, mass 0.057434868067502975; visual mesh filename=meshes/vis_vertebra_caudal_39.obj scale=1.0 1.0 1.0
- added link vertebra_caudal_40_link, mass 0.035911206156015396; visual mesh filename=meshes/vis_vertebra_caudal_40.obj scale=1.0 1.0 1.0
- added link vertebra_caudal_41_link, mass 0.024224260821938515; visual mesh filename=meshes/vis_vertebra_caudal_41.obj scale=1.0 1.0 1.0
- added link vertebra_caudal_42_link, mass 0.01687365211546421; visual mesh filename=meshes/vis_vertebra_caudal_42.obj scale=1.0 1.0 1.0
- added link vertebra_caudal_43_link, mass 0.015275629237294197; visual mesh filename=meshes/vis_vertebra_caudal_43.obj scale=1.0 1.0 1.0
- added link vertebra_caudal_44_link, mass 0.011179223656654358; visual mesh filename=meshes/vis_vertebra_caudal_44.obj scale=1.0 1.0 1.0
- link atlas_axis_link: geometry visual mesh filename=meshes/vis_atlas_axis.obj scale=1.0 1.0 1.0; visual mesh filename=meshes/vis_rib_cervical_01_L.obj scale=1.0 1.0 1.0
- link cranium_link: geometry visual mesh filename=meshes/vis_cranium.obj scale=1.0 1.0 1.0; visual mesh filename=meshes/vis_palette.obj scale=1.0 1.0 1.0
- link digit_01_a_L_link: geometry visual mesh filename=meshes/vis_digit_01_a_L.obj scale=1.0 1.0 1.0
- link digit_01_a_R_link: geometry visual mesh filename=meshes/vis_digit_01_a_R.obj scale=1.0 1.0 1.0
- link digit_01_b_L_link: geometry visual mesh filename=meshes/vis_digit_01_b_L.obj scale=1.0 1.0 1.0
- link digit_01_b_R_link: geometry visual mesh filename=meshes/vis_digit_01_b_R.obj scale=1.0 1.0 1.0
- link digit_01_c_L_link: geometry visual mesh filename=meshes/vis_digit_01_c_L.obj scale=1.0 1.0 1.0
- link digit_01_c_R_link: geometry visual mesh filename=meshes/vis_digit_01_c_R.obj scale=1.0 1.0 1.0
- link digit_02_a_L_link: geometry visual mesh filename=meshes/vis_digit_02_a_L.obj scale=1.0 1.0 1.0
- link digit_02_a_R_link: geometry visual mesh filename=meshes/vis_digit_02_a_R.obj scale=1.0 1.0 1.0
- link digit_02_b_L_link: geometry visual mesh filename=meshes/vis_digit_02_b_L.obj scale=1.0 1.0 1.0
- link digit_02_b_R_link: geometry visual mesh filename=meshes/vis_digit_02_b_R.obj scale=1.0 1.0 1.0
- link digit_02_c_L_link: geometry visual mesh filename=meshes/vis_digit_02_c_L.obj scale=1.0 1.0 1.0
- link digit_02_c_R_link: geometry visual mesh filename=meshes/vis_digit_02_c_R.obj scale=1.0 1.0 1.0
- link digit_02_d_L_link: geometry visual mesh filename=meshes/vis_digit_02_d_L.obj scale=1.0 1.0 1.0
- link digit_02_d_R_link: geometry visual mesh filename=meshes/vis_digit_02_d_R.obj scale=1.0 1.0 1.0
- link digit_03_a_L_link: geometry visual mesh filename=meshes/vis_digit_03_a_L.obj scale=1.0 1.0 1.0
- link digit_03_a_R_link: geometry visual mesh filename=meshes/vis_digit_03_a_R.obj scale=1.0 1.0 1.0
- link femur_L_link: geometry visual mesh filename=meshes/vis_femur_L.obj scale=1.0 1.0 1.0
- link femur_R_link: geometry visual mesh filename=meshes/vis_femur_R.obj scale=1.0 1.0 1.0
- link humerus_L_link: geometry visual mesh filename=meshes/vis_humerus_L.obj scale=1.0 1.0 1.0
- link humerus_R_link: geometry visual mesh filename=meshes/vis_humerus_R.obj scale=1.0 1.0 1.0
- link mandible_link: geometry visual mesh filename=meshes/vis_lower_teeth.obj scale=1.0 1.0 1.0; visual mesh filename=meshes/vis_mandible.obj scale=1.0 1.0 1.0
- link radius_L_link: geometry visual mesh filename=meshes/vis_radius_L.obj scale=1.0 1.0 1.0
- link radius_R_link: geometry visual mesh filename=meshes/vis_radius_R.obj scale=1.0 1.0 1.0
- link scapula_corcoid_L_link: geometry visual mesh filename=meshes/vis_scapula_corcoid_L.obj scale=1.0 1.0 1.0
- link scapula_corcoid_R_link: geometry visual mesh filename=meshes/vis_scapula_corcoid_R.obj scale=1.0 1.0 1.0
- link tarsometatarsus_L_link: geometry visual mesh filename=meshes/vis_tarsometatarsus_L.obj scale=1.0 1.0 1.0
- link tarsometatarsus_R_link: geometry visual mesh filename=meshes/vis_tarsometatarsus_R.obj scale=1.0 1.0 1.0
- link tibia_L_link: geometry visual mesh filename=meshes/vis_fibula_L.obj scale=1.0 1.0 1.0; visual mesh filename=meshes/vis_tibia_L.obj scale=1.0 1.0 1.0
- link tibia_R_link: geometry visual mesh filename=meshes/vis_fibula_R.obj scale=1.0 1.0 1.0; visual mesh filename=meshes/vis_tibia_R.obj scale=1.0 1.0 1.0
- link toe_01_a_L_link: geometry visual mesh filename=meshes/vis_toe_01_a_L.obj scale=1.0 1.0 1.0
- link toe_01_a_R_link: geometry visual mesh filename=meshes/vis_toe_01_a_R.obj scale=1.0 1.0 1.0
- link toe_01_b_L_link: geometry visual mesh filename=meshes/vis_toe_01_b_L.obj scale=1.0 1.0 1.0
- link toe_01_b_R_link: geometry visual mesh filename=meshes/vis_toe_01_b_R.obj scale=1.0 1.0 1.0
- link toe_01_c_L_link: geometry visual mesh filename=meshes/vis_toe_01_c_L.obj scale=1.0 1.0 1.0
- link toe_01_c_R_link: geometry visual mesh filename=meshes/vis_toe_01_c_R.obj scale=1.0 1.0 1.0
- link toe_02_a_L_link: geometry visual mesh filename=meshes/vis_toe_02_a_L.obj scale=1.0 1.0 1.0
- link toe_02_a_R_link: geometry visual mesh filename=meshes/vis_toe_02_a_R.obj scale=1.0 1.0 1.0
- link toe_02_b_L_link: geometry visual mesh filename=meshes/vis_toe_02_b_L.obj scale=1.0 1.0 1.0
- link toe_02_b_R_link: geometry visual mesh filename=meshes/vis_toe_02_b_R.obj scale=1.0 1.0 1.0
- link toe_02_c_L_link: geometry visual mesh filename=meshes/vis_toe_02_c_L.obj scale=1.0 1.0 1.0
- link toe_02_c_R_link: geometry visual mesh filename=meshes/vis_toe_02_c_R.obj scale=1.0 1.0 1.0
- link toe_03_a_L_link: geometry visual mesh filename=meshes/vis_toe_03_a_L.obj scale=1.0 1.0 1.0
- link toe_03_a_R_link: geometry visual mesh filename=meshes/vis_toe_03_a_R.obj scale=1.0 1.0 1.0
- link toe_03_b_L_link: geometry visual mesh filename=meshes/vis_toe_03_b_L.obj scale=1.0 1.0 1.0
- link toe_03_b_R_link: geometry visual mesh filename=meshes/vis_toe_03_b_R.obj scale=1.0 1.0 1.0
- link toe_03_c_L_link: geometry visual mesh filename=meshes/vis_toe_03_c_L.obj scale=1.0 1.0 1.0
- link toe_03_c_R_link: geometry visual mesh filename=meshes/vis_toe_03_c_R.obj scale=1.0 1.0 1.0
- link toe_03_d_L_link: geometry visual mesh filename=meshes/vis_toe_03_d_L.obj scale=1.0 1.0 1.0
- link toe_03_d_R_link: geometry visual mesh filename=meshes/vis_toe_03_d_R.obj scale=1.0 1.0 1.0
- link toe_04_a_L_link: geometry visual mesh filename=meshes/vis_toe_04_a_L.obj scale=1.0 1.0 1.0
- link toe_04_a_R_link: geometry visual mesh filename=meshes/vis_toe_04_a_R.obj scale=1.0 1.0 1.0
- link toe_04_b_L_link: geometry visual mesh filename=meshes/vis_toe_04_b_L.obj scale=1.0 1.0 1.0
- link toe_04_b_R_link: geometry visual mesh filename=meshes/vis_toe_04_b_R.obj scale=1.0 1.0 1.0
- link toe_04_c_L_link: geometry visual mesh filename=meshes/vis_toe_04_c_L.obj scale=1.0 1.0 1.0
- link toe_04_c_R_link: geometry visual mesh filename=meshes/vis_toe_04_c_R.obj scale=1.0 1.0 1.0
- link toe_04_d_L_link: geometry visual mesh filename=meshes/vis_toe_04_d_L.obj scale=1.0 1.0 1.0
- link toe_04_d_R_link: geometry visual mesh filename=meshes/vis_toe_04_d_R.obj scale=1.0 1.0 1.0
- link toe_04_e_L_link: geometry visual mesh filename=meshes/vis_toe_04_e_L.obj scale=1.0 1.0 1.0
- link toe_04_e_R_link: geometry visual mesh filename=meshes/vis_toe_04_e_R.obj scale=1.0 1.0 1.0
- link toe_05_a_L_link: geometry visual mesh filename=meshes/vis_toe_05_a_L.obj scale=1.0 1.0 1.0
- link toe_05_a_R_link: geometry visual mesh filename=meshes/vis_toe_05_a_R.obj scale=1.0 1.0 1.0
- link ulna_L_link: geometry visual mesh filename=meshes/vis_ulna_L.obj scale=1.0 1.0 1.0
- link ulna_R_link: geometry visual mesh filename=meshes/vis_ulna_R.obj scale=1.0 1.0 1.0
- link vertebra_caudal_00_link: geometry visual mesh filename=meshes/vis_gorgo_haemal_arch_01.obj scale=1.0 1.0 1.0; visual mesh filename=meshes/vis_vertebra_caudal_00.obj scale=1.0 1.0 1.0
- link vertebra_caudal_01_link: geometry visual mesh filename=meshes/vis_gorgo_haemal_arch_02.obj scale=1.0 1.0 1.0; visual mesh filename=meshes/vis_vertebra_caudal_01.obj scale=1.0 1.0 1.0
- link vertebra_caudal_02_link: geometry visual mesh filename=meshes/vis_gorgo_haemal_arch_03.obj scale=1.0 1.0 1.0; visual mesh filename=meshes/vis_vertebra_caudal_02.obj scale=1.0 1.0 1.0
- link vertebra_caudal_03_link: geometry visual mesh filename=meshes/vis_gorgo_haemal_arch_04.obj scale=1.0 1.0 1.0; visual mesh filename=meshes/vis_vertebra_caudal_03.obj scale=1.0 1.0 1.0
- link vertebra_caudal_04_link: geometry visual mesh filename=meshes/vis_gorgo_haemal_arch_05.obj scale=1.0 1.0 1.0; visual mesh filename=meshes/vis_vertebra_caudal_04.obj scale=1.0 1.0 1.0
- link vertebra_caudal_05_link: geometry visual mesh filename=meshes/vis_gorgo_haemal_arch_06.obj scale=1.0 1.0 1.0; visual mesh filename=meshes/vis_vertebra_caudal_05.obj scale=1.0 1.0 1.0
- link vertebra_caudal_06_link: geometry visual mesh filename=meshes/vis_gorgo_haemal_arch_07.obj scale=1.0 1.0 1.0; visual mesh filename=meshes/vis_vertebra_caudal_06.obj scale=1.0 1.0 1.0
- link vertebra_caudal_07_link: geometry visual mesh filename=meshes/vis_gorgo_haemal_arch_08.obj scale=1.0 1.0 1.0; visual mesh filename=meshes/vis_vertebra_caudal_07.obj scale=1.0 1.0 1.0
- link vertebra_caudal_08_link: geometry visual mesh filename=meshes/vis_gorgo_haemal_arch_09.obj scale=1.0 1.0 1.0; visual mesh filename=meshes/vis_vertebra_caudal_08.obj scale=1.0 1.0 1.0
- link vertebra_caudal_09_link: geometry visual mesh filename=meshes/vis_gorgo_haemal_arch_10.obj scale=1.0 1.0 1.0; visual mesh filename=meshes/vis_vertebra_caudal_09.obj scale=1.0 1.0 1.0
- link vertebra_caudal_10_link: geometry visual mesh filename=meshes/vis_gorgo_haemal_arch_11.obj scale=1.0 1.0 1.0; visual mesh filename=meshes/vis_vertebra_caudal_10.obj scale=1.0 1.0 1.0
- link vertebra_caudal_11_link: geometry visual mesh filename=meshes/vis_gorgo_haemal_arch_12.obj scale=1.0 1.0 1.0; visual mesh filename=meshes/vis_vertebra_caudal_11.obj scale=1.0 1.0 1.0
- link vertebra_caudal_12_link: geometry visual mesh filename=meshes/vis_gorgo_haemal_arch_13.obj scale=1.0 1.0 1.0; visual mesh filename=meshes/vis_vertebra_caudal_12.obj scale=1.0 1.0 1.0
- link vertebra_caudal_13_link: geometry visual mesh filename=meshes/vis_gorgo_haemal_arch_14.obj scale=1.0 1.0 1.0; visual mesh filename=meshes/vis_vertebra_caudal_13.obj scale=1.0 1.0 1.0
- link vertebra_caudal_14_link: geometry visual mesh filename=meshes/vis_gorgo_haemal_arch_15.obj scale=1.0 1.0 1.0; visual mesh filename=meshes/vis_vertebra_caudal_14.obj scale=1.0 1.0 1.0
- link vertebra_caudal_15_link: geometry visual mesh filename=meshes/vis_gorgo_haemal_arch_16.obj scale=1.0 1.0 1.0; visual mesh filename=meshes/vis_vertebra_caudal_15.obj scale=1.0 1.0 1.0
- link vertebra_caudal_16_link: geometry visual mesh filename=meshes/vis_gorgo_haemal_arch_17.obj scale=1.0 1.0 1.0; visual mesh filename=meshes/vis_vertebra_caudal_16.obj scale=1.0 1.0 1.0
- link vertebra_caudal_17_link: geometry visual mesh filename=meshes/vis_gorgo_haemal_arch_18.obj scale=1.0 1.0 1.0; visual mesh filename=meshes/vis_vertebra_caudal_17.obj scale=1.0 1.0 1.0
- link vertebra_caudal_18_link: geometry visual mesh filename=meshes/vis_gorgo_haemal_arch_19.obj scale=1.0 1.0 1.0; visual mesh filename=meshes/vis_vertebra_caudal_18.obj scale=1.0 1.0 1.0
- link vertebra_caudal_19_link: geometry visual mesh filename=meshes/vis_gorgo_haemal_arch_20.obj scale=1.0 1.0 1.0; visual mesh filename=meshes/vis_vertebra_caudal_19.obj scale=1.0 1.0 1.0
- link vertebra_caudal_20_link: geometry visual mesh filename=meshes/vis_gorgo_haemal_arch_21.obj scale=1.0 1.0 1.0; visual mesh filename=meshes/vis_vertebra_caudal_20.obj scale=1.0 1.0 1.0
- link vertebra_caudal_21_link: geometry visual mesh filename=meshes/vis_gorgo_haemal_arch_22.obj scale=1.0 1.0 1.0; visual mesh filename=meshes/vis_vertebra_caudal_21.obj scale=1.0 1.0 1.0
- link vertebra_caudal_22_link: geometry visual mesh filename=meshes/vis_gorgo_haemal_arch_23.obj scale=1.0 1.0 1.0; visual mesh filename=meshes/vis_vertebra_caudal_22.obj scale=1.0 1.0 1.0
- link vertebra_caudal_23_link: geometry visual mesh filename=meshes/vis_gorgo_haemal_arch_24.obj scale=1.0 1.0 1.0; visual mesh filename=meshes/vis_vertebra_caudal_23.obj scale=1.0 1.0 1.0
- link vertebra_caudal_24_link: geometry visual mesh filename=meshes/vis_gorgo_haemal_arch_25.obj scale=1.0 1.0 1.0; visual mesh filename=meshes/vis_vertebra_caudal_24.obj scale=1.0 1.0 1.0
- link vertebra_caudal_25_link: geometry visual mesh filename=meshes/vis_gorgo_haemal_arch_26.obj scale=1.0 1.0 1.0; visual mesh filename=meshes/vis_vertebra_caudal_25.obj scale=1.0 1.0 1.0
- link vertebra_cervical_01_link: geometry visual mesh filename=meshes/vis_rib_cervical_02_L.obj scale=1.0 1.0 1.0; visual mesh filename=meshes/vis_rib_cervical_02_R.obj scale=1.0 1.0 1.0
- link vertebra_cervical_02_link: geometry visual mesh filename=meshes/vis_rib_cervical_03_L.obj scale=1.0 1.0 1.0; visual mesh filename=meshes/vis_rib_cervical_03_R.obj scale=1.0 1.0 1.0
- link vertebra_cervical_03_link: geometry visual mesh filename=meshes/vis_rib_cervical_04_L.obj scale=1.0 1.0 1.0; visual mesh filename=meshes/vis_rib_cervical_04_R.obj scale=1.0 1.0 1.0
- link vertebra_cervical_04_link: geometry visual mesh filename=meshes/vis_rib_cervical_05_L.obj scale=1.0 1.0 1.0; visual mesh filename=meshes/vis_rib_cervical_05_R.obj scale=1.0 1.0 1.0
- link vertebra_cervical_05_link: geometry visual mesh filename=meshes/vis_rib_cervical_06_L.obj scale=1.0 1.0 1.0; visual mesh filename=meshes/vis_rib_cervical_06_R.obj scale=1.0 1.0 1.0
- link vertebra_cervical_06_link: geometry visual mesh filename=meshes/vis_rib_cervical_07_L.obj scale=1.0 1.0 1.0; visual mesh filename=meshes/vis_rib_cervical_07_R.obj scale=1.0 1.0 1.0
- link vertebra_cervical_07_link: geometry visual mesh filename=meshes/vis_rib_cervical_08_L.obj scale=1.0 1.0 1.0; visual mesh filename=meshes/vis_rib_cervical_08_R.obj scale=1.0 1.0 1.0
- link vertebra_cervical_08_link: geometry visual mesh filename=meshes/vis_rib_cervical_09_L.obj scale=1.0 1.0 1.0; visual mesh filename=meshes/vis_rib_cervical_09_R.obj scale=1.0 1.0 1.0
- link vertebra_cervical_09_link: geometry visual mesh filename=meshes/vis_rib_cervical_10_L.obj scale=1.0 1.0 1.0; visual mesh filename=meshes/vis_rib_cervical_10_R.obj scale=1.0 1.0 1.0
- link vertebra_dorsal_00_link: geometry visual mesh filename=meshes/vis_vertebra_dorsal_00.obj scale=1.0 1.0 1.0
- link vertebra_dorsal_01_link: geometry visual mesh filename=meshes/vis_rib_dorsal_01_L.obj scale=1.0 1.0 1.0; visual mesh filename=meshes/vis_rib_dorsal_01_R.obj scale=1.0 1.0 1.0
- link vertebra_dorsal_02_link: geometry visual mesh filename=meshes/vis_furcula.obj scale=1.0 1.0 1.0; visual mesh filename=meshes/vis_rib_dorsal_02_L.obj scale=1.0 1.0 1.0
- link vertebra_dorsal_03_link: geometry visual mesh filename=meshes/vis_rib_dorsal_03_L.obj scale=1.0 1.0 1.0; visual mesh filename=meshes/vis_rib_dorsal_03_R.obj scale=1.0 1.0 1.0
- link vertebra_dorsal_04_link: geometry visual mesh filename=meshes/vis_rib_dorsal_04_L.obj scale=1.0 1.0 1.0; visual mesh filename=meshes/vis_rib_dorsal_04_R.obj scale=1.0 1.0 1.0
- link vertebra_dorsal_05_link: geometry visual mesh filename=meshes/vis_gastralium_01_L.obj scale=1.0 1.0 1.0; visual mesh filename=meshes/vis_gastralium_01_R.obj scale=1.0 1.0 1.0
- link vertebra_dorsal_06_link: geometry visual mesh filename=meshes/vis_gastralium_03_L.obj scale=1.0 1.0 1.0; visual mesh filename=meshes/vis_gastralium_03_R.obj scale=1.0 1.0 1.0
- link vertebra_dorsal_07_link: geometry visual mesh filename=meshes/vis_gastralium_05_L.obj scale=1.0 1.0 1.0; visual mesh filename=meshes/vis_gastralium_05_R.obj scale=1.0 1.0 1.0
- link vertebra_dorsal_08_link: geometry visual mesh filename=meshes/vis_gastralium_07_L.obj scale=1.0 1.0 1.0; visual mesh filename=meshes/vis_gastralium_07_R.obj scale=1.0 1.0 1.0
- link vertebra_dorsal_09_link: geometry visual mesh filename=meshes/vis_gastralium_10_L.obj scale=1.0 1.0 1.0; visual mesh filename=meshes/vis_gastralium_10_R.obj scale=1.0 1.0 1.0
- link vertebra_dorsal_10_link: geometry visual mesh filename=meshes/vis_gastralium_12_L.obj scale=1.0 1.0 1.0; visual mesh filename=meshes/vis_gastralium_12_R.obj scale=1.0 1.0 1.0
- link vertebra_dorsal_11_link: geometry visual mesh filename=meshes/vis_rib_dorsal_11_L.obj scale=1.0 1.0 1.0; visual mesh filename=meshes/vis_rib_dorsal_11_R.obj scale=1.0 1.0 1.0
- link vertebra_dorsal_12_link: geometry visual mesh filename=meshes/vis_vertebra_dorsal_12.obj scale=1.0 1.0 1.0
- link vertebrae_sacral_link: geometry visual mesh filename=meshes/vis_ilium_L.obj scale=1.0 1.0 1.0; visual mesh filename=meshes/vis_ilium_R.obj scale=1.0 1.0 1.0
Joints:
- added joint vertebra_caudal_26_joint: type fixed, parent vertebra_caudal_25_link, child vertebra_caudal_26_link, origin xyz=-1.1396958043974337e-08 0.12284772843122482 -6.741020186495916e-09 rpy=0.0872664526104927 -0.0 0.0, axis 0.0 0.0 1.0, limit lower=1.0 upper=1.0 effort=100.0 velocity=1.0
- added joint vertebra_caudal_27_joint: type fixed, parent vertebra_caudal_26_link, child vertebra_caudal_27_link, origin xyz=-3.238782753101077e-08 0.1170744001865387 8.482263780251742e-09 rpy=-0.03490658476948738 -0.0 0.0, axis 0.0 0.0 1.0, limit lower=1.0 upper=1.0 effort=100.0 velocity=1.0
- added joint vertebra_caudal_28_joint: type fixed, parent vertebra_caudal_27_link, child vertebra_caudal_28_link, origin xyz=-2.5515602075643073e-08 0.10653021931648254 -1.3911666485455498e-08 rpy=0.01745329238474369 -0.0 0.0, axis 0.0 0.0 1.0, limit lower=1.0 upper=1.0 effort=100.0 velocity=1.0
- added joint vertebra_caudal_29_joint: type fixed, parent vertebra_caudal_28_link, child vertebra_caudal_29_link, origin xyz=-1.838031948864227e-08 0.11145378649234772 -5.123079915847484e-08 rpy=0.05235988274216652 -0.0 0.0, axis 0.0 0.0 1.0, limit lower=1.0 upper=1.0 effort=100.0 velocity=1.0
- added joint vertebra_caudal_30_joint: type fixed, parent vertebra_caudal_29_link, child vertebra_caudal_30_link, origin xyz=-1.6345827802410895e-08 0.09971961379051208 1.129853330894548e-07 rpy=0.01745329238474369 -0.0 0.0, axis 0.0 0.0 1.0, limit lower=1.0 upper=1.0 effort=100.0 velocity=1.0
- added joint vertebra_caudal_31_joint: type fixed, parent vertebra_caudal_30_link, child vertebra_caudal_31_link, origin xyz=-1.711174490992562e-08 0.0900387242436409 -6.582843781188785e-08 rpy=0.05235988274216652 -0.0 0.0, axis 0.0 0.0 1.0, limit lower=1.0 upper=1.0 effort=100.0 velocity=1.0
- added joint vertebra_caudal_32_joint: type fixed, parent vertebra_caudal_31_link, child vertebra_caudal_32_link, origin xyz=-2.6825375698535936e-08 0.08127997070550919 -1.17729825888091e-07 rpy=-0.01745329238474369 -0.0 0.0, axis 0.0 0.0 1.0, limit lower=1.0 upper=1.0 effort=100.0 velocity=1.0
- added joint vertebra_caudal_33_joint: type fixed, parent vertebra_caudal_32_link, child vertebra_caudal_33_link, origin xyz=-2.7043547845551075e-08 0.07476441562175751 4.5586949681819533e-07 rpy=0.06981316208839417 -0.0 0.0, axis 0.0 0.0 1.0, limit lower=1.0 upper=1.0 effort=100.0 velocity=1.0
- added joint vertebra_caudal_34_joint: type fixed, parent vertebra_caudal_33_link, child vertebra_caudal_34_link, origin xyz=-7.998536943887302e-09 0.07271556556224823 1.1359605878169532e-07 rpy=0.06981316208839417 -0.0 0.0, axis 0.0 0.0 1.0, limit lower=1.0 upper=1.0 effort=100.0 velocity=1.0
- added joint vertebra_caudal_35_joint: type fixed, parent vertebra_caudal_34_link, child vertebra_caudal_35_link, origin xyz=-3.205924414828587e-08 0.06442441791296005 -3.1073011541593587e-07 rpy=-0.03490658476948738 -0.0 0.0, axis 0.0 0.0 1.0, limit lower=1.0 upper=1.0 effort=100.0 velocity=1.0
- added joint vertebra_caudal_36_joint: type fixed, parent vertebra_caudal_35_link, child vertebra_caudal_36_link, origin xyz=-1.7920257278092322e-08 0.07024165242910385 -5.766185395827961e-08 rpy=0.0 -0.0 0.0, axis 0.0 0.0 1.0, limit lower=1.0 upper=1.0 effort=100.0 velocity=1.0
- added joint vertebra_caudal_37_joint: type fixed, parent vertebra_caudal_36_link, child vertebra_caudal_37_link, origin xyz=-1.3081617566967907e-08 0.06583874672651291 -5.02694383897051e-08 rpy=0.01745329238474369 -0.0 0.0, axis 0.0 0.0 1.0, limit lower=1.0 upper=1.0 effort=100.0 velocity=1.0
- added joint vertebra_caudal_38_joint: type fixed, parent vertebra_caudal_37_link, child vertebra_caudal_38_link, origin xyz=8.14770118040542e-09 0.052238158881664276 9.126684119564743e-08 rpy=0.05235988274216652 -0.0 0.0, axis 0.0 0.0 1.0, limit lower=1.0 upper=1.0 effort=100.0 velocity=1.0
- added joint vertebra_caudal_39_joint: type fixed, parent vertebra_caudal_38_link, child vertebra_caudal_39_link, origin xyz=-8.406338736222096e-09 0.0513455830514431 2.032991233136272e-07 rpy=-0.01745329238474369 -0.0 0.0, axis 0.0 0.0 1.0, limit lower=1.0 upper=1.0 effort=100.0 velocity=1.0
- added joint vertebra_caudal_40_joint: type fixed, parent vertebra_caudal_39_link, child vertebra_caudal_40_link, origin xyz=3.6381067047841498e-09 0.04671191796660423 -2.4374821805395186e-07 rpy=-0.01745329238474369 -0.0 0.0, axis 0.0 0.0 1.0, limit lower=1.0 upper=1.0 effort=100.0 velocity=1.0
- added joint vertebra_caudal_41_joint: type fixed, parent vertebra_caudal_40_link, child vertebra_caudal_41_link, origin xyz=-2.20197371447739e-08 0.040036316961050034 9.877827977788911e-08 rpy=0.05235988274216652 -0.0 0.0, axis 0.0 0.0 1.0, limit lower=1.0 upper=1.0 effort=100.0 velocity=1.0
- added joint vertebra_caudal_42_joint: type fixed, parent vertebra_caudal_41_link, child vertebra_caudal_42_link, origin xyz=-3.5276372045700555e-08 0.03419726714491844 2.92717373895357e-07 rpy=0.10471975803375244 -0.0 0.0, axis 0.0 0.0 1.0, limit lower=1.0 upper=1.0 effort=100.0 velocity=1.0
- added joint vertebra_caudal_43_joint: type fixed, parent vertebra_caudal_42_link, child vertebra_caudal_43_link, origin xyz=1.9819879071292235e-09 0.033248838037252426 2.7475061870063655e-07 rpy=-0.05235988274216652 -0.0 0.0, axis 0.0 0.0 1.0, limit lower=1.0 upper=1.0 effort=100.0 velocity=1.0
- added joint vertebra_caudal_44_joint: type fixed, parent vertebra_caudal_43_link, child vertebra_caudal_44_link, origin xyz=-4.39769820559377e-09 0.034847550094127655 2.6313898615626385e-07 rpy=0.0 -0.0 0.0, axis 0.0 0.0 1.0, limit lower=1.0 upper=1.0 effort=100.0 velocity=1.0
