Commit message: Add a world joint and make URDF-to-MuJoCo include a free-joint.

File: assets/trex.urdf (robot description, URDF)
Before this commit: robot stan_t_rex, 133 links, 132 joints
Links:
- added link world
Joints:
- added joint joint_world_to_sacrum: type floating, parent world, child link_vertebrae_sacral, origin xyz=0.0 0.0 0.0 rpy=0.0 0.0 0.0

Commit message: Add generated collision capsules

File: assets/trex.urdf (robot description, URDF)
Before this commit: robot stan_t_rex, 134 links, 133 joints
Links:
- link link_cranium: geometry collision capsule length=0.8695043963660251 radius=0.581242829812658; visual mesh filename=meshes/cranium.obj scale=1.0 1.0 1.0
- link link_tarsometatarsus_left: geometry collision capsule length=0.41519850814619663 radius=0.19651473310014886; visual mesh filename=meshes/tarsometatarsus_left.obj scale=1.0 1.0 1.0
- link link_tarsometatarsus_right: geometry collision capsule length=0.4204948843738786 radius=0.1961608907276992; visual mesh filename=meshes/tarsometatarsus_right.obj scale=1.0 1.0 1.0
- link link_toe_01_a_left: geometry collision capsule length=0.08988255569011548 radius=0.03951409872299168; visual mesh filename=meshes/toe_01_a_left.obj scale=1.0 1.0 1.0
- link link_toe_01_a_right: geometry collision capsule length=0.09893455985318592 radius=0.03732940617741446; visual mesh filename=meshes/toe_01_a_right.obj scale=1.0 1.0 1.0
- link link_toe_01_b_left: geometry collision capsule length=0.0942721084625497 radius=0.03330442243607323; visual mesh filename=meshes/toe_01_b_left.obj scale=1.0 1.0 1.0
- link link_toe_01_b_right: geometry collision capsule length=0.09516667710736464 radius=0.03334301962394471; visual mesh filename=meshes/toe_01_b_right.obj scale=1.0 1.0 1.0
- link link_toe_01_c_left: geometry collision capsule length=0.11646185731690266 radius=0.028488092598899933; visual mesh filename=meshes/toe_01_c_left.obj scale=1.0 1.0 1.0
- link link_toe_01_c_right: geometry collision capsule length=0.11762773866236595 radius=0.028361971155339005; visual mesh filename=meshes/toe_01_c_right.obj scale=1.0 1.0 1.0
- link link_toe_02_a_left: geometry collision capsule length=0.14257939263190905 radius=0.0926854536553942; visual mesh filename=meshes/toe_02_a_left.obj scale=1.0 1.0 1.0
- link link_toe_02_a_right: geometry collision capsule length=0.15566837064808223 radius=0.09163016597659768; visual mesh filename=meshes/toe_02_a_right.obj scale=1.0 1.0 1.0
- link link_toe_02_b_left: geometry collision capsule length=0.12196642476969599 radius=0.06065632895616454; visual mesh filename=meshes/toe_02_b_left.obj scale=1.0 1.0 1.0
- link link_toe_02_b_right: geometry collision capsule length=0.12242484819020395 radius=0.06061798605116905; visual mesh filename=meshes/toe_02_b_right.obj scale=1.0 1.0 1.0
- link link_toe_02_c_left: geometry collision capsule length=0.12288707956706639 radius=0.039512617255557714; visual mesh filename=meshes/toe_02_c_left.obj scale=1.0 1.0 1.0
- link link_toe_02_c_right: geometry collision capsule length=0.12294026303933266 radius=0.039399990199069014; visual mesh filename=meshes/toe_02_c_right.obj scale=1.0 1.0 1.0
- link link_toe_03_a_left: geometry collision capsule length=0.16787624710414262 radius=0.07777879407395766; visual mesh filename=meshes/toe_03_a_left.obj scale=1.0 1.0 1.0
- link link_toe_03_a_right: geometry collision capsule length=0.1405684110670034 radius=0.08176208834178365; visual mesh filename=meshes/toe_03_a_right.obj scale=1.0 1.0 1.0
- link link_toe_03_b_left: geometry collision capsule length=0.10035344882787786 radius=0.06566556311126061; visual mesh filename=meshes/toe_03_b_left.obj scale=1.0 1.0 1.0
- link link_toe_03_b_right: geometry collision capsule length=0.09450222574578866 radius=0.06559828439833719; visual mesh filename=meshes/toe_03_b_right.obj scale=1.0 1.0 1.0
- link link_toe_03_c_left: geometry collision capsule length=0.10566321087561746 radius=0.05444940328396773; visual mesh filename=meshes/toe_03_c_left.obj scale=1.0 1.0 1.0
- link link_toe_03_c_right: geometry collision capsule length=0.11406065576824265 radius=0.05345803952836962; visual mesh filename=meshes/toe_03_c_right.obj scale=1.0 1.0 1.0
- link link_toe_03_d_left: geometry collision capsule length=0.09157804589719945 radius=0.044418045416528947; visual mesh filename=meshes/toe_03_d_left.obj scale=1.0 1.0 1.0
- link link_toe_03_d_right: geometry collision capsule length=0.091712280583625 radius=0.044167939953435466; visual mesh filename=meshes/toe_03_d_right.obj scale=1.0 1.0 1.0
- link link_toe_04_a_left: geometry collision capsule length=0.10676444880197003 radius=0.08497498248746185; visual mesh filename=meshes/toe_04_a_left.obj scale=1.0 1.0 1.0
- link link_toe_04_a_right: geometry collision capsule length=0.11027858747108531 radius=0.08375986623981806; visual mesh filename=meshes/toe_04_a_right.obj scale=1.0 1.0 1.0
- link link_toe_04_b_left: geometry collision capsule length=0.033077137372364854 radius=0.06793914134164114; visual mesh filename=meshes/toe_04_b_left.obj scale=1.0 1.0 1.0
- link link_toe_04_b_right: geometry collision capsule length=0.03632944859853013 radius=0.06745278523661603; visual mesh filename=meshes/toe_04_b_right.obj scale=1.0 1.0 1.0
- link link_toe_04_c_left: geometry collision capsule length=0.018744423767272096 radius=0.06916729803631674; visual mesh filename=meshes/toe_04_c_left.obj scale=1.0 1.0 1.0
- link link_toe_04_c_right: geometry collision capsule length=0.017802768072510265 radius=0.06918167522884996; visual mesh filename=meshes/toe_04_c_right.obj scale=1.0 1.0 1.0
- link link_toe_04_d_left: geometry collision capsule length=0.04059161497193256 radius=0.05098557207538333; visual mesh filename=meshes/toe_04_d_left.obj scale=1.0 1.0 1.0
- link link_toe_04_d_right: geometry collision capsule length=0.0356556278711672 radius=0.05271432167834396; visual mesh filename=meshes/toe_04_d_right.obj scale=1.0 1.0 1.0
- link link_toe_04_e_left: geometry collision capsule length=0.10766211313301463 radius=0.03412965105910412; visual mesh filename=meshes/toe_04_e_left.obj scale=1.0 1.0 1.0
- link link_toe_04_e_right: geometry collision capsule length=0.10766263767787751 radius=0.03425266752740769; visual mesh filename=meshes/toe_04_e_right.obj scale=1.0 1.0 1.0
- link link_toe_05_a_left: geometry collision capsule length=0.21809880203269266 radius=0.04379949280824006; visual mesh filename=meshes/toe_05_a_left.obj scale=1.0 1.0 1.0
- link link_toe_05_a_right: geometry collision capsule length=0.2170583023377086 radius=0.04352986689920897; visual mesh filename=meshes/toe_05_a_right.obj scale=1.0 1.0 1.0
- link link_vertebra_caudal_00: geometry collision capsule length=1.6918844633055186 radius=0.42923432534998474; visual mesh filename=meshes/gorgo_haemal_arch_01.obj scale=1.0 1.0 1.0
- link link_vertebra_caudal_10: geometry collision capsule length=1.805692624304582 radius=0.28502244374714775; visual mesh filename=meshes/gorgo_haemal_arch_11.obj scale=1.0 1.0 1.0
- link link_vertebra_caudal_24: geometry collision capsule length=0.8922383681107176 radius=0.10190880523404405; visual mesh filename=meshes/gorgo_haemal_arch_25.obj scale=1.0 1.0 1.0
- link link_vertebra_caudal_34: geometry collision capsule length=0.5273449769907109 radius=0.029396737590706355; visual mesh filename=meshes/vertebra_caudal_34.obj scale=1.0 1.0 1.0
- link link_vertebra_cervical_09: geometry collision capsule length=1.1825671370789907 radius=0.3624312979938864; visual mesh filename=meshes/rib_cervical_10_left.obj scale=1.0 1.0 1.0
- link link_vertebra_dorsal_04: geometry collision capsule length=0.6576748982466329 radius=0.6968781662471596; visual mesh filename=meshes/rib_dorsal_04_left.obj scale=1.0 1.0 1.0
- link link_vertebra_dorsal_08: geometry collision capsule length=0.5032856994006939 radius=0.702693982515512; visual mesh filename=meshes/gastralium_07_left.obj scale=1.0 1.0 1.0
- link link_vertebra_dorsal_12: geometry collision capsule length=0.7054000668756726 radius=0.607780892590496; visual mesh filename=meshes/vertebra_dorsal_12.obj scale=1.0 1.0 1.0
- link link_vertebrae_sacral: geometry collision capsule length=0.4099513036342905 radius=1.0419539665370925; visual mesh filename=meshes/ilium_left.obj scale=1.0 1.0 1.0

Commit message: Refine generated foot collision capsules

File: assets/trex.urdf (robot description, URDF)
Before this commit: robot stan_t_rex, 134 links, 133 joints
Links:
- link link_tarsometatarsus_left: geometry collision capsule length=0.47171971564338344 radius=0.12477937318185695; collision capsule length=0.5016941505600471 radius=0.11062523225218085
- link link_tarsometatarsus_right: geometry collision capsule length=0.48937356140745336 radius=0.12401791437270072; collision capsule length=0.5047673317768125 radius=0.11257100065460349
- link link_toe_01_a_left: geometry visual mesh filename=meshes/toe_01_a_left.obj scale=1.0 1.0 1.0
- link link_toe_01_a_right: geometry visual mesh filename=meshes/toe_01_a_right.obj scale=1.0 1.0 1.0
- link link_toe_05_a_left: geometry visual mesh filename=meshes/toe_05_a_left.obj scale=1.0 1.0 1.0
- link link_toe_05_a_right: geometry visual mesh filename=meshes/toe_05_a_right.obj scale=1.0 1.0 1.0

Commit message: Replace pelvis collision capsule with femurs

File: assets/trex.urdf (robot description, URDF)
Before this commit: robot stan_t_rex, 134 links, 133 joints
Links:
- link link_femur_left: geometry collision capsule length=1.1038630702242727 radius=0.2161464748064217; visual mesh filename=meshes/femur_left.obj scale=1.0 1.0 1.0
- link link_femur_right: geometry collision capsule length=1.1135891817381736 radius=0.21451770675865311; visual mesh filename=meshes/femur_right.obj scale=1.0 1.0 1.0
- link link_vertebrae_sacral: geometry visual mesh filename=meshes/ilium_left.obj scale=1.0 1.0 1.0; visual mesh filename=meshes/ilium_right.obj scale=1.0 1.0 1.0

Commit message: Add linked hip adduction DOFs

File: assets/trex.urdf (robot description, URDF)
Before this commit: robot stan_t_rex, 134 links, 133 joints
Links:
- added link link_hip_adduction_left
- added link link_hip_adduction_right
Joints:
- added joint joint_hip_adduction_left: type revolute, parent link_vertebrae_sacral, child link_hip_adduction_left, origin xyz=0.01719667762517929 -0.2207697629928589 -0.24924658238887787 rpy=3.141592502593994 -0.0 0.27925267815589905, axis 1.0 0.0 0.0, limit lower=-0.7853981633974483 upper=0.7853981633974483 effort=100.0 velocity=1.0
- added joint joint_hip_adduction_right: type revolute, parent link_vertebrae_sacral, child link_hip_adduction_right, origin xyz=0.0171966552734375 -0.2207697629928589 0.2492464929819107 rpy=-3.141592502593994 -0.0 0.27925267815589905, axis 1.0 0.0 0.0, limit lower=-0.7853981633974483 upper=0.7853981633974483 effort=100.0 velocity=1.0
- joint joint_femur_left: origin xyz=0.01719667762517929 -0.2207697629928589 -0.24924658238887787 rpy=3.141592502593994 -0.0 0.27925267815589905 -> xyz=0.0 0.0 0.0 rpy=0.0 0.0 0.0; parent link_vertebrae_sacral -> link_hip_adduction_left
- joint joint_femur_right: origin xyz=0.0171966552734375 -0.2207697629928589 0.2492464929819107 rpy=-3.141592502593994 -0.0 0.27925267815589905 -> xyz=0.0 0.0 0.0 rpy=0.0 0.0 0.0; parent link_vertebrae_sacral -> link_hip_adduction_right

Commit message: Limit hip adduction range

File: assets/trex.urdf (robot description, URDF)
Before this commit: robot stan_t_rex, 136 links, 135 joints
Joints:
- joint joint_hip_adduction_left: limit lower=-0.7853981633974483 upper=0.7853981633974483 effort=100.0 velocity=1.0 -> lower=-0.2617993877991494 upper=0.7853981633974483 effort=100.0 velocity=1.0
- joint joint_hip_adduction_right: limit lower=-0.7853981633974483 upper=0.7853981633974483 effort=100.0 velocity=1.0 -> lower=-0.7853981633974483 upper=0.2617993877991494 effort=100.0 velocity=1.0

Commit message: Refine caudal tail joints and capsules

File: assets/trex.urdf (robot description, URDF)
Before this commit: robot stan_t_rex, 136 links, 135 joints
Links:
- link link_vertebra_caudal_00: geometry visual mesh filename=meshes/gorgo_haemal_arch_01.obj scale=1.0 1.0 1.0; visual mesh filename=meshes/vertebra_caudal_00.obj scale=1.0 1.0 1.0
- link link_vertebra_caudal_09: geometry collision capsule length=1.6918844633055186 radius=0.4292343253499847; visual mesh filename=meshes/gorgo_haemal_arch_10.obj scale=1.0 1.0 1.0
- link link_vertebra_caudal_10: geometry visual mesh filename=meshes/gorgo_haemal_arch_11.obj scale=1.0 1.0 1.0; visual mesh filename=meshes/vertebra_caudal_10.obj scale=1.0 1.0 1.0
- link link_vertebra_caudal_23: geometry collision capsule length=1.8056926243045799 radius=0.28502244374714786; visual mesh filename=meshes/gorgo_haemal_arch_24.obj scale=1.0 1.0 1.0
- link link_vertebra_caudal_24: geometry visual mesh filename=meshes/gorgo_haemal_arch_25.obj scale=1.0 1.0 1.0; visual mesh filename=meshes/vertebra_caudal_24.obj scale=1.0 1.0 1.0
- link link_vertebra_caudal_33: geometry collision capsule length=0.8922383681107187 radius=0.101908805234044; visual mesh filename=meshes/gorgo_haemal_arch_34.obj scale=1.0 1.0 1.0
- link link_vertebra_caudal_34: geometry visual mesh filename=meshes/vertebra_caudal_34.obj scale=1.0 1.0 1.0
- link link_vertebra_caudal_44: geometry collision capsule length=0.5273449769907105 radius=0.029396737590706566; visual mesh filename=meshes/vertebra_caudal_44.obj scale=1.0 1.0 1.0
Joints:
- joint joint_vertebra_caudal_03: limit lower=1.0 upper=1.0 effort=100.0 velocity=1.0 -> lower=-0.3490658503988659 upper=0.3490658503988659 effort=100.0 velocity=1.0; type fixed -> revolute
- joint joint_vertebra_caudal_10: axis 0.0 0.0 1.0 -> 1.0 0.0 0.0; limit lower=-1.3490658503988659 upper=1.3490658503988659 effort=100.0 velocity=1.0 -> lower=-0.3490658503988659 upper=0.3490658503988659 effort=100.0 velocity=1.0
- joint joint_vertebra_caudal_11: limit lower=1.0 upper=1.0 effort=100.0 velocity=1.0 -> lower=-0.3490658503988659 upper=0.3490658503988659 effort=100.0 velocity=1.0; type fixed -> revolute
- joint joint_vertebra_caudal_25: limit lower=1.0 upper=1.0 effort=100.0 velocity=1.0 -> lower=-0.3490658503988659 upper=0.3490658503988659 effort=100.0 velocity=1.0; type fixed -> revolute
- joint joint_vertebra_caudal_34: limit lower=1.0 upper=1.0 effort=100.0 velocity=1.0 -> lower=-0.3490658503988659 upper=0.3490658503988659 effort=100.0 velocity=1.0; type fixed -> revolute
